File: sheet/sheet.sch (KiCad schematic (older format))
At the start: 44 parts

Commit message: Normalize component name case and underscores
Parts:
- removed R?: R-0,125W, symbol R-0,125W
- added R?: R_0,125W, symbol R_0,125W
- C?: value C-EL -> C_EL; symbol C-EL -> C_EL
- C?: value C-POL -> C_Pol; symbol C-POL -> C_Pol
- C?: value C-EL-NONPOL -> C_EL_Nonpol; symbol C-EL-NONPOL -> C_EL_Nonpol
- C?: value C_VAR -> C_Var; symbol C_VAR -> C_Var
- C?: value C_TRIM -> C_Trim; symbol C_TRIM -> C_Trim
- FU?: value FUSE -> Fuse; symbol FUSE -> Fuse
- FU?: value POLYFUSE -> Polyfuse; symbol POLYFUSE -> Polyfuse
- GB?: value BATTERY -> Battery; symbol BATTERY -> Battery
- GB?: value BATTERY2 -> Battery2; symbol BATTERY2 -> Battery2
- L?: value L3_FERRITE -> L3_Ferrite; symbol L3_FERRITE -> L3_Ferrite
- L?: value L_FERRITE -> L_Ferrite; symbol L_FERRITE -> L_Ferrite
- R?: value R_TRIM -> R_Trim; symbol R_TRIM -> R_Trim
- R?: value R_VARIABLE -> R_Var; symbol R_VARIABLE -> R_Var
- RK?: value THERMISTOR -> Thermistor; symbol THERMISTOR -> Thermistor
- VD?: value DIODE -> Diode; symbol DIODE -> Diode
- VD?: value SCHOTTKY_DIODE -> Schottky_Diode; symbol SCHOTTKY_DIODE -> Schottky_Diode
- VT?: value NMOS_CIRCLE -> NMOS_Circle; symbol NMOS_CIRCLE -> NMOS_Circle
- VT?: value PMOS_CIRCLE -> PMOS_Circle; symbol PMOS_CIRCLE -> PMOS_Circle
- VT?: value NPN_CIRCLE -> NPN_Circle; symbol NPN_CIRCLE -> NPN_Circle
- VT?: value PNP_CIRCLE -> PNP_Circle; symbol PNP_CIRCLE -> PNP_Circle
Changed lines of the file:
@@
 LIBS:semiconductors
 LIBS:switches
+LIBS:sheet-cache
 EELAYER 25 0
 EELAYER END
@@
 $EndComp
 $Comp
-L C-EL C?
+L C_EL C?
 U 1 1 55D8CAA7
 P 1850 1000
 F 0 "C?" V 2005 1000 50  0000 C CNN
-F 1 "C-EL" V 1700 1000 50  0000 C CNN
+F 1 "C_EL" V 1700 1000 50  0000 C CNN
 F 2 "" H 1850 1000 60  0000 C CNN
 F 3 "" H 1850 1000 60  0000 C CNN
@@
 $EndComp
 $Comp
-L FUSE FU?
+L Fuse FU?
 U 1 1 55D8CAF1
 P 1650 2050
 F 0 "FU?" H 1650 2150 50  0000 C CNN
-F 1 "FUSE" H 1650 1950 50  0000 C CNN
+F 1 "Fuse" H 1650 1950 50  0000 C CNN
 F 2 "" H 1700 1850 60  0000 C CNN
 F 3 "" H 1650 2050 60  0000 C CNN
@@
 $EndComp
 $Comp
-L L3_FERRITE L?
+L L3_Ferrite L?
 U 1 1 55D8CC6C
 P 1950 3500
 F 0 "L?" H 1955 3650 50  0000 C CNN
-F 1 "L3_FERRITE" H 1975 3425 50  0000 C CNN
+F 1 "L3_Ferrite" H 1975 3425 50  0000 C CNN
 F 2 "" H 1950 3500 60  0000 C CNN
 F 3 "" H 1950 3500 60  0000 C CNN
@@
 $EndComp
 $Comp
-L L_FERRITE L?
+L L_Ferrite L?
 U 1 1 55D8CCBD
 P 1150 3500
 F 0 "L?" H 1155 3650 50  0000 C CNN
-F 1 "L_FERRITE" H 1150 3425 50  0000 C CNN
+F 1 "L_Ferrite" H 1150 3425 50  0000 C CNN
 F 2 "" H 1075 3500 60  0000 C CNN
 F 3 "" H 1075 3500 60  0000 C CNN
@@
 $EndComp
 $Comp
-L POLYFUSE FU?
+L Polyfuse FU?
 U 1 1 55D8CD66
 P 1050 2050
 F 0 "FU?" H 1055 2200 50  0000 C CNN
-F 1 "POLYFUSE" H 1050 1850 50  0000 C CNN
+F 1 "Polyfuse" H 1050 1850 50  0000 C CNN
 F 2 "" H 1050 2050 60  0000 C CNN
 F 3 "" H 1050 2050 60  0000 C CNN
@@
 $EndComp
 $Comp
-L THERMISTOR RK?
+L Thermistor RK?
 U 1 1 55D8CDF1
 P 1050 2550
 F 0 "RK?" H 1055 2700 50  0000 C CNN
-F 1 "THERMISTOR" H 1050 2350 50  0000 C CNN
+F 1 "Thermistor" H 1050 2350 50  0000 C CNN
 F 2 "" H 1050 2550 60  0000 C CNN
 F 3 "" H 1050 2550 60  0000 C CNN
@@
 $EndComp
 $Comp
-L R_TRIM R?
+L R_Trim R?
 U 1 1 55D8CE2C
 P 1050 3050
 F 0 "R?" H 1055 3200 50  0000 C CNN
-F 1 "R_TRIM" H 1050 2900 50  0000 C CNN
+F 1 "R_Trim" H 1050 2900 50  0000 C CNN
 F 2 "" H 1050 3050 60  0000 C CNN
 F 3 "" H 1050 3050 60  0000 C CNN
@@
 $EndComp
 $Comp
-L R_VARIABLE R?
+L R_Var R?
 U 1 1 55D8CE7D
 P 1650 3050
 F 0 "R?" H 1650 2850 50  0000 C CNN
-F 1 "R_VARIABLE" H 1650 2950 50  0000 C CNN
+F 1 "R_Var" H 1650 2950 50  0000 C CNN
 F 2 "" H 1650 3050 60  0000 C CNN
 F 3 "" H 1650 3050 60  0000 C CNN
@@
 Semicoductors
 $Comp
-L DIODE VD?
+L Diode VD?
 U 1 1 55D9AECA
 P 3050 2200
 F 0 "VD?" H 3050 2100 60  0000 C CNN
-F 1 "DIODE" H 3050 2300 60  0000 C CNN
+F 1 "Diode" H 3050 2300 60  0000 C CNN
 F 2 "" H 3050 2200 60  0000 C CNN
 F 3 "" H 3050 2200 60  0000 C CNN
@@
 $EndComp
 $Comp
-L SCHOTTKY_DIODE VD?
+L Schottky_Diode VD?
 U 1 1 55D9AF25
 P 3700 2200
 F 0 "VD?" H 3700 2100 60  0000 C CNN
-F 1 "SCHOTTKY_DIODE" H 3700 2300 60  0000 C CNN
+F 1 "Schottky_Diode" H 3700 2300 60  0000 C CNN
 F 2 "" H 3700 2200 60  0000 C CNN
 F 3 "" H 3700 2200 60  0000 C CNN
@@
 Regulators
 $Comp
-L BATTERY GB?
+L Battery GB?
 U 1 1 55D9BEA9
 P 5850 2750
 F 0 "GB?" V 5975 2750 60  0000 C CNN
-F 1 "BATTERY" V 5725 2750 60  0000 C CNN
+F 1 "Battery" V 5725 2750 60  0000 C CNN
 F 2 "" H 5850 2750 60  0000 C CNN
 F 3 "" H 5850 2750 60  0000 C CNN
@@
 $EndComp
 $Comp
-L BATTERY2 GB?
+L Battery2 GB?
 U 1 1 55D9BF58
 P 6300 2850
 F 0 "GB?" V 6425 2840 60  0000 C CNN
-F 1 "BATTERY2" V 6175 2850 60  0000 C CNN
+F 1 "Battery2" V 6175 2850 60  0000 C CNN
 F 2 "" H 6300 2850 60  0000 C CNN
 F 3 "" H 6300 2850 60  0000 C CNN
@@
 $EndComp
 $Comp
-L NMOS_CIRCLE VT?
+L NMOS_Circle VT?
 U 1 1 55DAE0AB
 P 4300 3200
 F 0 "VT?" H 4400 3050 60  0000 R CNN
-F 1 "NMOS_CIRCLE" H 4650 3400 60  0000 R CNN
+F 1 "NMOS_Circle" H 4650 3400 60  0000 R CNN
 F 2 "" H 4275 3225 60  0000 C CNN
 F 3 "" H 4275 3225 60  0000 C CNN
@@
 $EndComp
 $Comp
-L PMOS_CIRCLE VT?
+L PMOS_Circle VT?
 U 1 1 55DAE216
 P 5000 3200
 F 0 "VT?" H 5100 3050 60  0000 R CNN
-F 1 "PMOS_CIRCLE" H 5350 3400 60  0000 R CNN
+F 1 "PMOS_Circle" H 5350 3400 60  0000 R CNN
 F 2 "" H 4975 3225 60  0000 C CNN
 F 3 "" H 4975 3225 60  0000 C CNN
@@
 $EndComp
 $Comp
-L NPN_CIRCLE VT?
+L NPN_Circle VT?
 U 1 1 55DB069D
 P 3050 3150
 F 0 "VT?" H 3025 3000 60  0000 R CNN
-F 1 "NPN_CIRCLE" H 3050 3300 60  0000 R CNN
+F 1 "NPN_Circle" H 3050 3300 60  0000 R CNN
 F 2 "" H 3050 3150 60  0000 C CNN
 F 3 "" H 3050 3150 60  0000 C CNN
@@
 $EndComp
 $Comp
-L PNP_CIRCLE VT?
+L PNP_Circle VT?
 U 1 1 55DB0714
 P 3700 3150
 F 0 "VT?" H 3675 3000 60  0000 R CNN
-F 1 "PNP_CIRCLE" H 3700 3300 60  0000 R CNN
+F 1 "PNP_Circle" H 3700 3300 60  0000 R CNN
 F 2 "" H 3700 3150 60  0000 C CNN
 F 3 "" H 3700 3150 60  0000 C CNN
@@
 $EndComp
 $Comp
-L C-POL C?
+L C_Pol C?
 U 1 1 55DB600C
 P 1400 1000
 F 0 "C?" V 1555 1000 50  0000 C CNN
-F 1 "C-POL" V 1250 1000 50  0000 C CNN
+F 1 "C_Pol" V 1250 1000 50  0000 C CNN
 F 2 "" H 1400 1000 60  0000 C CNN
 F 3 "" H 1400 1000 60  0000 C CNN
@@
 $EndComp
 $Comp
-L C-EL-NONPOL C?
+L C_EL_Nonpol C?
 U 1 1 55DB73DF
 P 2300 1000
 F 0 "C?" V 2455 1000 50  0000 C CNN
-F 1 "C-EL-NONPOL" V 2150 1000 50  0000 C CNN
+F 1 "C_EL_Nonpol" V 2150 1000 50  0000 C CNN
 F 2 "" H 2300 1000 60  0000 C CNN
 F 3 "" H 2300 1000 60  0000 C CNN
@@
 $EndComp
 $Comp
-L R-0,125W R?
-U 1 1 55DB7D86
-P 2250 2550
-F 0 "R?" V 2355 2550 50  0000 C CNN
-F 1 "R-0,125W" V 2150 2550 50  0000 C CNN
-F 2 "" H 2250 2550 60  0000 C CNN
-F 3 "" H 2250 2550 60  0000 C CNN
-	1    2250 2550
-	0    -1   -1   0
-$EndComp
-$Comp
-L C_VAR C?
+L C_Var C?
 U 1 1 55DBBA9B
 P 950 1500
 F 0 "C?" V 1105 1500 50  0000 C CNN
-F 1 "C_VAR" V 800 1500 50  0000 C CNN
+F 1 "C_Var" V 800 1500 50  0000 C CNN
 F 2 "" H 950 1500 60  0000 C CNN
 F 3 "" H 950 1500 60  0000 C CNN
@@
 $EndComp
 $Comp
-L C_TRIM C?
+L C_Trim C?
 U 1 1 55DC565E
 P 1400 1500
 F 0 "C?" V 1555 1500 50  0000 C CNN
-F 1 "C_TRIM" V 1250 1500 50  0000 C CNN
+F 1 "C_Trim" V 1250 1500 50  0000 C CNN
 F 2 "" H 1400 1500 60  0000 C CNN
 F 3 "" H 1400 1500 60  0000 C CNN
@@
 	1    0    0    -1
 $EndComp
+$Comp
+L R_0,125W R?
+U 1 1 55DBA828
+P 2250 2050
+F 0 "R?" V 2355 2050 50  0000 C CNN
+F 1 "R_0,125W" V 2150 2050 50  0000 C CNN
+F 2 "" H 2250 2050 60  0000 C CNN
+F 3 "" H 2250 2050 60  0000 C CNN
+	1    2250 2050
+	0    1    1    0
+$EndComp
 $EndSCHEMATC

Commit message: Correct transistors' arrows
Parts:
- added L?: L3, symbol L3
Changed lines of the file:
@@
 U 1 1 55D9F494
 P 950 4450
-F 0 "HL?" H 850 4600 60  0000 C CNN
-F 1 "LED" H 1075 4600 60  0000 C CNN
+F 0 "HL?" H 950 4300 60  0000 C CNN
+F 1 "LED" H 950 4700 60  0000 C CNN
 F 2 "" H 950 4450 60  0000 C CNN
 F 3 "" H 950 4450 60  0000 C CNN
@@
 	0    1    1    0
 $EndComp
+$Comp
+L L3 L?
+U 1 1 55E02239
+P 1950 3850
+F 0 "L?" H 1950 3975 50  0000 C CNN
+F 1 "L3" H 1950 3775 50  0000 C CNN
+F 2 "" H 1950 3850 60  0000 C CNN
+F 3 "" H 1950 3850 60  0000 C CNN
+	1    1950 3850
+	1    0    0    -1
+$EndComp
 $EndSCHEMATC

Commit message: Add Zener, tunel, backward diodes, varicap, dynistor, DIAC
Parts:
- added VD?: Zener_Diode, symbol Zener_Diode
- added VD?: Zener_Diode_Double-anode, symbol Zener_Diode_Double-anode
- added VD?: Varicap, symbol Varicap
- added VD?: Tunnel_Diode, symbol Tunnel_Diode
- added VD?: Backward_Diode, symbol Backward_Diode
Other:
- moved on the sheet: DA?, HL?, VT?, XP?, XS?
Changed lines of the file:
@@
 L Diode VD?
 U 1 1 55D9AECA
-P 3050 2200
-F 0 "VD?" H 3050 2100 60  0000 C CNN
-F 1 "Diode" H 3050 2300 60  0000 C CNN
-F 2 "" H 3050 2200 60  0000 C CNN
-F 3 "" H 3050 2200 60  0000 C CNN
-	1    3050 2200
+P 3050 2600
+F 0 "VD?" H 3050 2500 60  0000 C CNN
+F 1 "Diode" H 3050 2700 60  0000 C CNN
+F 2 "" H 3050 2600 60  0000 C CNN
+F 3 "" H 3050 2600 60  0000 C CNN
+	1    3050 2600
 	1    0    0    -1
 $EndComp
@@
 L Schottky_Diode VD?
 U 1 1 55D9AF25
-P 3700 2200
-F 0 "VD?" H 3700 2100 60  0000 C CNN
-F 1 "Schottky_Diode" H 3700 2300 60  0000 C CNN
-F 2 "" H 3700 2200 60  0000 C CNN
-F 3 "" H 3700 2200 60  0000 C CNN
-	1    3700 2200
+P 3700 2600
+F 0 "VD?" H 3700 2500 60  0000 C CNN
+F 1 "Schottky_Diode" H 3700 2700 60  0000 C CNN
+F 2 "" H 3700 2600 60  0000 C CNN
+F 3 "" H 3700 2600 60  0000 C CNN
+	1    3700 2600
 	1    0    0    -1
 $EndComp
@@
 L NMOS VT?
 U 1 1 55D9AF68
-P 4300 2700
-F 0 "VT?" H 4425 2525 60  0000 R CNN
-F 1 "NMOS" H 4475 2875 60  0000 R CNN
-F 2 "" H 4300 2700 60  0000 C CNN
-F 3 "" H 4300 2700 60  0000 C CNN
-	1    4300 2700
+P 4300 3600
+F 0 "VT?" H 4425 3425 60  0000 R CNN
+F 1 "NMOS" H 4475 3775 60  0000 R CNN
+F 2 "" H 4300 3600 60  0000 C CNN
+F 3 "" H 4300 3600 60  0000 C CNN
+	1    4300 3600
 	1    0    0    -1
 $EndComp
@@
 L PMOS VT?
 U 1 1 55D9AFE5
-P 5000 2700
-F 0 "VT?" H 5125 2525 60  0000 R CNN
-F 1 "PMOS" H 5175 2875 60  0000 R CNN
-F 2 "" H 5000 2700 60  0000 C CNN
-F 3 "" H 5000 2700 60  0000 C CNN
-	1    5000 2700
+P 5000 3600
+F 0 "VT?" H 5125 3425 60  0000 R CNN
+F 1 "PMOS" H 5175 3775 60  0000 R CNN
+F 2 "" H 5000 3600 60  0000 C CNN
+F 3 "" H 5000 3600 60  0000 C CNN
+	1    5000 3600
 	1    0    0    -1
 $EndComp
@@
 L NPN VT?
 U 1 1 55D9B10B
-P 3050 2650
-F 0 "VT?" H 3025 2500 60  0000 R CNN
-F 1 "NPN" H 3050 2800 60  0000 R CNN
-F 2 "" H 3050 2650 60  0000 C CNN
-F 3 "" H 3050 2650 60  0000 C CNN
-	1    3050 2650
+P 3050 3550
+F 0 "VT?" H 3025 3400 60  0000 R CNN
+F 1 "NPN" H 3050 3700 60  0000 R CNN
+F 2 "" H 3050 3550 60  0000 C CNN
+F 3 "" H 3050 3550 60  0000 C CNN
+	1    3050 3550
 	1    0    0    -1
 $EndComp
@@
 L PNP VT?
 U 1 1 55D9B160
-P 3700 2650
-F 0 "VT?" H 3675 2500 60  0000 R CNN
-F 1 "PNP" H 3700 2800 60  0000 R CNN
-F 2 "" H 3700 2650 60  0000 C CNN
-F 3 "" H 3700 2650 60  0000 C CNN
-	1    3700 2650
+P 3700 3550
+F 0 "VT?" H 3675 3400 60  0000 R CNN
+F 1 "PNP" H 3700 3700 60  0000 R CNN
+F 2 "" H 3700 3550 60  0000 C CNN
+F 3 "" H 3700 3550 60  0000 C CNN
+	1    3700 3550
 	1    0    0    -1
 $EndComp
@@
 L REG2 DA?
 U 1 1 55D9B4E5
-P 5200 1850
-F 0 "DA?" H 4935 2100 60  0000 C CNN
-F 1 "REG2" H 5350 2100 60  0000 C CNN
-F 2 "" H 5200 1850 60  0000 C CNN
-F 3 "" H 5200 1850 60  0000 C CNN
-	1    5200 1850
+P 5150 1850
+F 0 "DA?" H 4885 2100 60  0000 C CNN
+F 1 "REG2" H 5300 2100 60  0000 C CNN
+F 2 "" H 5150 1850 60  0000 C CNN
+F 3 "" H 5150 1850 60  0000 C CNN
+	1    5150 1850
 	1    0    0    -1
 $EndComp
@@
 L LED HL?
 U 1 1 55D9F494
-P 950 4450
-F 0 "HL?" H 950 4300 60  0000 C CNN
-F 1 "LED" H 950 4700 60  0000 C CNN
-F 2 "" H 950 4450 60  0000 C CNN
-F 3 "" H 950 4450 60  0000 C CNN
-	1    950  4450
-	1    0    0    -1
-$EndComp
-Text Notes 800  4100 0    60   ~ 0
+P 950 5600
+F 0 "HL?" H 950 5450 60  0000 C CNN
+F 1 "LED" H 950 5850 60  0000 C CNN
+F 2 "" H 950 5600 60  0000 C CNN
+F 3 "" H 950 5600 60  0000 C CNN
+	1    950  5600
+	1    0    0    -1
+$EndComp
+Text Notes 800  5250 0    60   ~ 0
 Indicators
 $Comp
 L CONN_02_F XS?
 U 1 1 55DA0C94
-P 2850 4450
-F 0 "XS?" H 3100 4550 60  0000 C CNN
-F 1 "CONN_02_F" H 3200 4250 60  0001 C CNN
-F 2 "" H 2850 4450 60  0000 C CNN
-F 3 "" H 2850 4450 60  0000 C CNN
-	1    2850 4450
+P 2850 5600
+F 0 "XS?" H 3100 5700 60  0000 C CNN
+F 1 "CONN_02_F" H 3200 5400 60  0001 C CNN
+F 2 "" H 2850 5600 60  0000 C CNN
+F 3 "" H 2850 5600 60  0000 C CNN
+	1    2850 5600
 	1    0    0    -1
 $EndComp
@@
 L CONN_02_M XP?
 U 1 1 55DA0E2F
-P 3650 4450
-F 0 "XP?" H 3900 4550 60  0000 C CNN
-F 1 "CONN_02_M" H 4000 4250 60  0001 C CNN
-F 2 "" H 3650 4450 60  0000 C CNN
-F 3 "" H 3650 4450 60  0000 C CNN
-	1    3650 4450
-	1    0    0    -1
-$EndComp
-Text Notes 2850 4100 0    60   ~ 0
+P 3650 5600
+F 0 "XP?" H 3900 5700 60  0000 C CNN
+F 1 "CONN_02_M" H 4000 5400 60  0001 C CNN
+F 2 "" H 3650 5600 60  0000 C CNN
+F 3 "" H 3650 5600 60  0000 C CNN
+	1    3650 5600
+	1    0    0    -1
+$EndComp
+Text Notes 2850 5250 0    60   ~ 0
 Connectors
 $Comp
 L PAD XS?
 U 1 1 55DA139F
-P 2850 4900
-F 0 "XS?" H 3100 5000 60  0000 C CNN
-F 1 "PAD" H 3100 4800 60  0000 C CNN
-F 2 "" H 2850 4900 60  0000 C CNN
-F 3 "" H 2850 4900 60  0000 C CNN
-	1    2850 4900
+P 2850 6050
+F 0 "XS?" H 3100 6150 60  0000 C CNN
+F 1 "PAD" H 3100 5950 60  0000 C CNN
+F 2 "" H 2850 6050 60  0000 C CNN
+F 3 "" H 2850 6050 60  0000 C CNN
+	1    2850 6050
 	1    0    0    -1
 $EndComp
@@
 L NMOS_Circle VT?
 U 1 1 55DAE0AB
-P 4300 3200
-F 0 "VT?" H 4400 3050 60  0000 R CNN
-F 1 "NMOS_Circle" H 4650 3400 60  0000 R CNN
-F 2 "" H 4275 3225 60  0000 C CNN
-F 3 "" H 4275 3225 60  0000 C CNN
-	1    4300 3200
+P 4300 4100
+F 0 "VT?" H 4400 3950 60  0000 R CNN
+F 1 "NMOS_Circle" H 4650 4300 60  0000 R CNN
+F 2 "" H 4275 4125 60  0000 C CNN
+F 3 "" H 4275 4125 60  0000 C CNN
+	1    4300 4100
 	1    0    0    -1
 $EndComp
@@
 L PMOS_Circle VT?
 U 1 1 55DAE216
-P 5000 3200
-F 0 "VT?" H 5100 3050 60  0000 R CNN
-F 1 "PMOS_Circle" H 5350 3400 60  0000 R CNN
-F 2 "" H 4975 3225 60  0000 C CNN
-F 3 "" H 4975 3225 60  0000 C CNN
-	1    5000 3200
+P 5000 4100
+F 0 "VT?" H 5100 3950 60  0000 R CNN
+F 1 "PMOS_Circle" H 5350 4300 60  0000 R CNN
+F 2 "" H 4975 4125 60  0000 C CNN
+F 3 "" H 4975 4125 60  0000 C CNN
+	1    5000 4100
 	1    0    0    -1
 $EndComp
@@
 L NPN_Circle VT?
 U 1 1 55DB069D
-P 3050 3150
-F 0 "VT?" H 3025 3000 60  0000 R CNN
-F 1 "NPN_Circle" H 3050 3300 60  0000 R CNN
-F 2 "" H 3050 3150 60  0000 C CNN
-F 3 "" H 3050 3150 60  0000 C CNN
-	1    3050 3150
+P 3050 4050
+F 0 "VT?" H 3025 3900 60  0000 R CNN
+F 1 "NPN_Circle" H 3050 4200 60  0000 R CNN
+F 2 "" H 3050 4050 60  0000 C CNN
+F 3 "" H 3050 4050 60  0000 C CNN
+	1    3050 4050
 	1    0    0    -1
 $EndComp
@@
 L PNP_Circle VT?
 U 1 1 55DB0714
-P 3700 3150
-F 0 "VT?" H 3675 3000 60  0000 R CNN
-F 1 "PNP_Circle" H 3700 3300 60  0000 R CNN
-F 2 "" H 3700 3150 60  0000 C CNN
-F 3 "" H 3700 3150 60  0000 C CNN
-	1    3700 3150
+P 3700 4050
+F 0 "VT?" H 3675 3900 60  0000 R CNN
+F 1 "PNP_Circle" H 3700 4200 60  0000 R CNN
+F 2 "" H 3700 4050 60  0000 C CNN
+F 3 "" H 3700 4050 60  0000 C CNN
+	1    3700 4050
 	1    0    0    -1
 $EndComp
@@
 	1    0    0    -1
 $EndComp
+$Comp
+L Zener_Diode VD?
+U 1 1 55E13EB1
+P 3050 3050
+F 0 "VD?" H 3050 2950 60  0000 C CNN
+F 1 "Zener_Diode" H 3050 3150 60  0000 C CNN
+F 2 "" H 3050 3050 60  0000 C CNN
+F 3 "" H 3050 3050 60  0000 C CNN
+	1    3050 3050
+	1    0    0    -1
+$EndComp
+$Comp
+L Zener_Diode_Double-anode VD?
+U 1 1 55E14A30
+P 4050 3050
+F 0 "VD?" H 4050 2950 60  0000 C CNN
+F 1 "Zener_Diode_Double-anode" H 4050 3150 60  0000 C CNN
+F 2 "" H 4000 3050 60  0000 C CNN
+F 3 "" H 4000 3050 60  0000 C CNN
+	1    4050 3050
+	1    0    0    -1
+$EndComp
+$Comp
+L Varicap VD?
+U 1 1 55E164B2
+P 5100 3050
+F 0 "VD?" H 5100 2950 60  0000 C CNN
+F 1 "Varicap" H 5100 3150 60  0000 C CNN
+F 2 "" H 5050 3050 60  0000 C CNN
+F 3 "" H 5050 3050 60  0000 C CNN
+	1    5100 3050
+	1    0    0    -1
+$EndComp
+$Comp
+L Tunnel_Diode VD?
+U 1 1 55E18AD5
+P 4400 2600
+F 0 "VD?" H 4400 2500 60  0000 C CNN
+F 1 "Tunnel_Diode" H 4400 2700 60  0000 C CNN
+F 2 "" H 4400 2600 60  0000 C CNN
+F 3 "" H 4400 2600 60  0000 C CNN
+	1    4400 2600
+	1    0    0    -1
+$EndComp
+$Comp
+L Backward_Diode VD?
+U 1 1 55E1BCCD
+P 5050 2600
+F 0 "VD?" H 5050 2500 60  0000 C CNN
+F 1 "Backward_Diode" H 5050 2700 60  0000 C CNN
+F 2 "" H 5050 2600 60  0000 C CNN
+F 3 "" H 5050 2600 60  0000 C CNN
+	1    5050 2600
+	1    0    0    -1
+$EndComp
