File: sheet/sheet.sch (KiCad schematic (older format))
At the start: 50 parts

Commit message: Added AGT, SCR, TRIC
Parts:
- added VS?: DIAC, symbol DIAC
- added VS?: Dynistor, symbol Dynistor
- added VS?: TRIAC, symbol TRIAC
- added VS?: Thyristor_Anode, symbol Thyristor_Anode
- added VS?: Thyristor_Cathode, symbol Thyristor_Cathode
Other:
- moved on the sheet: VT?, XP?, XS?
Changed lines of the file:
@@
 L NMOS VT?
 U 1 1 55D9AF68
-P 4300 3600
-F 0 "VT?" H 4425 3425 60  0000 R CNN
-F 1 "NMOS" H 4475 3775 60  0000 R CNN
-F 2 "" H 4300 3600 60  0000 C CNN
-F 3 "" H 4300 3600 60  0000 C CNN
-	1    4300 3600
+P 4300 4800
+F 0 "VT?" H 4425 4625 60  0000 R CNN
+F 1 "NMOS" H 4475 4975 60  0000 R CNN
+F 2 "" H 4300 4800 60  0000 C CNN
+F 3 "" H 4300 4800 60  0000 C CNN
+	1    4300 4800
 	1    0    0    -1
 $EndComp
@@
 L PMOS VT?
 U 1 1 55D9AFE5
-P 5000 3600
-F 0 "VT?" H 5125 3425 60  0000 R CNN
-F 1 "PMOS" H 5175 3775 60  0000 R CNN
-F 2 "" H 5000 3600 60  0000 C CNN
-F 3 "" H 5000 3600 60  0000 C CNN
-	1    5000 3600
+P 5000 4800
+F 0 "VT?" H 5125 4625 60  0000 R CNN
+F 1 "PMOS" H 5175 4975 60  0000 R CNN
+F 2 "" H 5000 4800 60  0000 C CNN
+F 3 "" H 5000 4800 60  0000 C CNN
+	1    5000 4800
 	1    0    0    -1
 $EndComp
@@
 L NPN VT?
 U 1 1 55D9B10B
-P 3050 3550
-F 0 "VT?" H 3025 3400 60  0000 R CNN
-F 1 "NPN" H 3050 3700 60  0000 R CNN
-F 2 "" H 3050 3550 60  0000 C CNN
-F 3 "" H 3050 3550 60  0000 C CNN
-	1    3050 3550
+P 3050 4750
+F 0 "VT?" H 3025 4600 60  0000 R CNN
+F 1 "NPN" H 3050 4900 60  0000 R CNN
+F 2 "" H 3050 4750 60  0000 C CNN
+F 3 "" H 3050 4750 60  0000 C CNN
+	1    3050 4750
 	1    0    0    -1
 $EndComp
@@
 L PNP VT?
 U 1 1 55D9B160
-P 3700 3550
-F 0 "VT?" H 3675 3400 60  0000 R CNN
-F 1 "PNP" H 3700 3700 60  0000 R CNN
-F 2 "" H 3700 3550 60  0000 C CNN
-F 3 "" H 3700 3550 60  0000 C CNN
-	1    3700 3550
+P 3700 4750
+F 0 "VT?" H 3675 4600 60  0000 R CNN
+F 1 "PNP" H 3700 4900 60  0000 R CNN
+F 2 "" H 3700 4750 60  0000 C CNN
+F 3 "" H 3700 4750 60  0000 C CNN
+	1    3700 4750
 	1    0    0    -1
 $EndComp
@@
 L CONN_02_F XS?
 U 1 1 55DA0C94
-P 2850 5600
-F 0 "XS?" H 3100 5700 60  0000 C CNN
-F 1 "CONN_02_F" H 3200 5400 60  0001 C CNN
-F 2 "" H 2850 5600 60  0000 C CNN
-F 3 "" H 2850 5600 60  0000 C CNN
-	1    2850 5600
+P 2850 5950
+F 0 "XS?" H 3100 6050 60  0000 C CNN
+F 1 "CONN_02_F" H 3200 5750 60  0001 C CNN
+F 2 "" H 2850 5950 60  0000 C CNN
+F 3 "" H 2850 5950 60  0000 C CNN
+	1    2850 5950
 	1    0    0    -1
 $EndComp
@@
 L CONN_02_M XP?
 U 1 1 55DA0E2F
-P 3650 5600
-F 0 "XP?" H 3900 5700 60  0000 C CNN
-F 1 "CONN_02_M" H 4000 5400 60  0001 C CNN
-F 2 "" H 3650 5600 60  0000 C CNN
-F 3 "" H 3650 5600 60  0000 C CNN
-	1    3650 5600
-	1    0    0    -1
-$EndComp
-Text Notes 2850 5250 0    60   ~ 0
+P 3650 5950
+F 0 "XP?" H 3900 6050 60  0000 C CNN
+F 1 "CONN_02_M" H 4000 5750 60  0001 C CNN
+F 2 "" H 3650 5950 60  0000 C CNN
+F 3 "" H 3650 5950 60  0000 C CNN
+	1    3650 5950
+	1    0    0    -1
+$EndComp
+Text Notes 2850 5600 0    60   ~ 0
 Connectors
 $Comp
 L PAD XS?
 U 1 1 55DA139F
-P 2850 6050
-F 0 "XS?" H 3100 6150 60  0000 C CNN
-F 1 "PAD" H 3100 5950 60  0000 C CNN
-F 2 "" H 2850 6050 60  0000 C CNN
-F 3 "" H 2850 6050 60  0000 C CNN
-	1    2850 6050
+P 2850 6400
+F 0 "XS?" H 3100 6500 60  0000 C CNN
+F 1 "PAD" H 3100 6300 60  0000 C CNN
+F 2 "" H 2850 6400 60  0000 C CNN
+F 3 "" H 2850 6400 60  0000 C CNN
+	1    2850 6400
 	1    0    0    -1
 $EndComp
@@
 L NMOS_Circle VT?
 U 1 1 55DAE0AB
-P 4300 4100
-F 0 "VT?" H 4400 3950 60  0000 R CNN
-F 1 "NMOS_Circle" H 4650 4300 60  0000 R CNN
-F 2 "" H 4275 4125 60  0000 C CNN
-F 3 "" H 4275 4125 60  0000 C CNN
-	1    4300 4100
+P 4300 5300
+F 0 "VT?" H 4400 5150 60  0000 R CNN
+F 1 "NMOS_Circle" H 4650 5500 60  0000 R CNN
+F 2 "" H 4275 5325 60  0000 C CNN
+F 3 "" H 4275 5325 60  0000 C CNN
+	1    4300 5300
 	1    0    0    -1
 $EndComp
@@
 L PMOS_Circle VT?
 U 1 1 55DAE216
-P 5000 4100
-F 0 "VT?" H 5100 3950 60  0000 R CNN
-F 1 "PMOS_Circle" H 5350 4300 60  0000 R CNN
-F 2 "" H 4975 4125 60  0000 C CNN
-F 3 "" H 4975 4125 60  0000 C CNN
-	1    5000 4100
+P 5000 5300
+F 0 "VT?" H 5100 5150 60  0000 R CNN
+F 1 "PMOS_Circle" H 5350 5500 60  0000 R CNN
+F 2 "" H 4975 5325 60  0000 C CNN
+F 3 "" H 4975 5325 60  0000 C CNN
+	1    5000 5300
 	1    0    0    -1
 $EndComp
@@
 L NPN_Circle VT?
 U 1 1 55DB069D
-P 3050 4050
-F 0 "VT?" H 3025 3900 60  0000 R CNN
-F 1 "NPN_Circle" H 3050 4200 60  0000 R CNN
-F 2 "" H 3050 4050 60  0000 C CNN
-F 3 "" H 3050 4050 60  0000 C CNN
-	1    3050 4050
+P 3050 5250
+F 0 "VT?" H 3025 5100 60  0000 R CNN
+F 1 "NPN_Circle" H 3050 5400 60  0000 R CNN
+F 2 "" H 3050 5250 60  0000 C CNN
+F 3 "" H 3050 5250 60  0000 C CNN
+	1    3050 5250
 	1    0    0    -1
 $EndComp
@@
 L PNP_Circle VT?
 U 1 1 55DB0714
-P 3700 4050
-F 0 "VT?" H 3675 3900 60  0000 R CNN
-F 1 "PNP_Circle" H 3700 4200 60  0000 R CNN
-F 2 "" H 3700 4050 60  0000 C CNN
-F 3 "" H 3700 4050 60  0000 C CNN
-	1    3700 4050
+P 3700 5250
+F 0 "VT?" H 3675 5100 60  0000 R CNN
+F 1 "PNP_Circle" H 3700 5400 60  0000 R CNN
+F 2 "" H 3700 5250 60  0000 C CNN
+F 3 "" H 3700 5250 60  0000 C CNN
+	1    3700 5250
 	1    0    0    -1
 $EndComp
@@
 L Zener_Diode_Double-anode VD?
 U 1 1 55E14A30
-P 4050 3050
-F 0 "VD?" H 4050 2950 60  0000 C CNN
-F 1 "Zener_Diode_Double-anode" H 4050 3150 60  0000 C CNN
-F 2 "" H 4000 3050 60  0000 C CNN
-F 3 "" H 4000 3050 60  0000 C CNN
-	1    4050 3050
+P 4100 3050
+F 0 "VD?" H 4100 2950 60  0000 C CNN
+F 1 "Zener_Diode_Double-anode" H 4100 3150 60  0000 C CNN
+F 2 "" H 4050 3050 60  0000 C CNN
+F 3 "" H 4050 3050 60  0000 C CNN
+	1    4100 3050
 	1    0    0    -1
 $EndComp
@@
 L Varicap VD?
 U 1 1 55E164B2
-P 5100 3050
-F 0 "VD?" H 5100 2950 60  0000 C CNN
-F 1 "Varicap" H 5100 3150 60  0000 C CNN
-F 2 "" H 5050 3050 60  0000 C CNN
-F 3 "" H 5050 3050 60  0000 C CNN
-	1    5100 3050
+P 5150 3050
+F 0 "VD?" H 5150 2950 60  0000 C CNN
+F 1 "Varicap" H 5150 3150 60  0000 C CNN
+F 2 "" H 5100 3050 60  0000 C CNN
+F 3 "" H 5100 3050 60  0000 C CNN
+	1    5150 3050
 	1    0    0    -1
 $EndComp
@@
 L Backward_Diode VD?
 U 1 1 55E1BCCD
-P 5050 2600
-F 0 "VD?" H 5050 2500 60  0000 C CNN
-F 1 "Backward_Diode" H 5050 2700 60  0000 C CNN
-F 2 "" H 5050 2600 60  0000 C CNN
-F 3 "" H 5050 2600 60  0000 C CNN
-	1    5050 2600
-	1    0    0    -1
-$EndComp
+P 5100 2600
+F 0 "VD?" H 5100 2500 60  0000 C CNN
+F 1 "Backward_Diode" H 5100 2700 60  0000 C CNN
+F 2 "" H 5100 2600 60  0000 C CNN
+F 3 "" H 5100 2600 60  0000 C CNN
+	1    5100 2600
+	1    0    0    -1
+$EndComp
+$Comp
+L DIAC VS?
+U 1 1 55E1F7D3
+P 3500 3500
+F 0 "VS?" H 3500 3325 60  0000 C CNN
+F 1 "DIAC" H 3500 3675 60  0000 C CNN
+F 2 "" H 3500 3450 60  0000 C CNN
+F 3 "" H 3500 3450 60  0000 C CNN
+	1    3500 3500
+	1    0    0    -1
+$EndComp
+$Comp
+L Dynistor VS?
+U 1 1 55E1F8C7
+P 3050 3500
+F 0 "VS?" H 3050 3400 60  0000 C CNN
+F 1 "Dynistor" H 3050 3600 60  0000 C CNN
+F 2 "" H 3050 3500 60  0000 C CNN
+F 3 "" H 3050 3500 60  0000 C CNN
+	1    3050 3500
+	1    0    0    -1
+$EndComp
+$Comp
+L TRIAC VS?
+U 1 1 55E1FAE8
+P 5100 3450
+F 0 "VS?" H 5100 3275 60  0000 C CNN
+F 1 "TRIAC" H 5100 3625 60  0000 C CNN
+F 2 "" H 5100 3400 60  0000 C CNN
+F 3 "" H 5100 3400 60  0000 C CNN
+	1    5100 3450
+	1    0    0    -1
+$EndComp
+$Comp
+L Thyristor_Anode VS?
+U 1 1 55E1FC03
+P 4600 3500
+F 0 "VS?" H 4600 3375 60  0000 C CNN
+F 1 "Thyristor_Anode" H 4600 3600 60  0000 C CNN
+F 2 "" H 4600 3500 60  0000 C CNN
+F 3 "" H 4600 3500 60  0000 C CNN
+	1    4600 3500
+	1    0    0    -1
+$EndComp
+$Comp
+L Thyristor_Cathode VS?
+U 1 1 55E1FCF5
+P 4000 3500
+F 0 "VS?" H 4000 3375 60  0000 C CNN
+F 1 "Thyristor_Cathode" H 4000 3700 60  0000 C CNN
+F 2 "" H 4000 3500 60  0000 C CNN
+F 3 "" H 4000 3500 60  0000 C CNN
+	1    4000 3500
+	1    0    0    -1
+$EndComp

Commit message: Add jfets, rename mosfets
Parts:
- removed VT?: NMOS, symbol NMOS
- removed VT?: PMOS, symbol PMOS
- removed VT?: NMOS_Circle, symbol NMOS_Circle
- removed VT?: PMOS_Circle, symbol PMOS_Circle
- added VT?: NJFET_Circle, symbol NJFET_Circle
- added VT?: NJFET, symbol NJFET
- added VT?: PJFET_Circle, symbol PJFET_Circle
- added VT?: PJFET, symbol PJFET
- added VT?: NMOSFET, symbol NMOSFET
- added VT?: NMOSFET_Circle, symbol NMOSFET_Circle
- added VT?: PMOSFET, symbol PMOSFET
- added VT?: PMOSFET_Circle, symbol PMOSFET_Circle
- added VT?: PMOSFET_DE, symbol PMOSFET_DE
- added VT?: PMOSFET_DE_Circle, symbol PMOSFET_DE_Circle
- added VT?: NMOSFET_DE, symbol NMOSFET_DE
- added VT?: NMOSFET_DE_Circle, symbol NMOSFET_DE_Circle
Other:
- moved on the sheet: VT?, XP?, XS?
Changed lines of the file:
@@
-$EndComp
-$Comp
-L NMOS VT?
-U 1 1 55D9AF68
-P 4300 4800
-F 0 "VT?" H 4425 4625 60  0000 R CNN
-F 1 "NMOS" H 4475 4975 60  0000 R CNN
-F 2 "" H 4300 4800 60  0000 C CNN
-F 3 "" H 4300 4800 60  0000 C CNN
-	1    4300 4800
-	1    0    0    -1
-$EndComp
-$Comp
-L PMOS VT?
-U 1 1 55D9AFE5
-P 5000 4800
-F 0 "VT?" H 5125 4625 60  0000 R CNN
-F 1 "PMOS" H 5175 4975 60  0000 R CNN
-F 2 "" H 5000 4800 60  0000 C CNN
-F 3 "" H 5000 4800 60  0000 C CNN
-	1    5000 4800
-	1    0    0    -1
 $EndComp
 $Comp
 L NPN VT?
 U 1 1 55D9B10B
-P 3050 4750
-F 0 "VT?" H 3025 4600 60  0000 R CNN
-F 1 "NPN" H 3050 4900 60  0000 R CNN
-F 2 "" H 3050 4750 60  0000 C CNN
-F 3 "" H 3050 4750 60  0000 C CNN
-	1    3050 4750
+P 3050 4000
+F 0 "VT?" H 3025 3850 60  0000 R CNN
+F 1 "NPN" H 3050 4150 60  0000 R CNN
+F 2 "" H 3050 4000 60  0000 C CNN
+F 3 "" H 3050 4000 60  0000 C CNN
+	1    3050 4000
 	1    0    0    -1
 $EndComp
@@
 L PNP VT?
 U 1 1 55D9B160
-P 3700 4750
-F 0 "VT?" H 3675 4600 60  0000 R CNN
-F 1 "PNP" H 3700 4900 60  0000 R CNN
-F 2 "" H 3700 4750 60  0000 C CNN
-F 3 "" H 3700 4750 60  0000 C CNN
-	1    3700 4750
+P 3700 4000
+F 0 "VT?" H 3675 3850 60  0000 R CNN
+F 1 "PNP" H 3700 4150 60  0000 R CNN
+F 2 "" H 3700 4000 60  0000 C CNN
+F 3 "" H 3700 4000 60  0000 C CNN
+	1    3700 4000
 	1    0    0    -1
 $EndComp
@@
 L CONN_02_F XS?
 U 1 1 55DA0C94
-P 2850 5950
-F 0 "XS?" H 3100 6050 60  0000 C CNN
-F 1 "CONN_02_F" H 3200 5750 60  0001 C CNN
-F 2 "" H 2850 5950 60  0000 C CNN
-F 3 "" H 2850 5950 60  0000 C CNN
-	1    2850 5950
+P 2850 6300
+F 0 "XS?" H 3100 6400 60  0000 C CNN
+F 1 "CONN_02_F" H 3200 6100 60  0001 C CNN
+F 2 "" H 2850 6300 60  0000 C CNN
+F 3 "" H 2850 6300 60  0000 C CNN
+	1    2850 6300
 	1    0    0    -1
 $EndComp
@@
 L CONN_02_M XP?
 U 1 1 55DA0E2F
-P 3650 5950
-F 0 "XP?" H 3900 6050 60  0000 C CNN
-F 1 "CONN_02_M" H 4000 5750 60  0001 C CNN
-F 2 "" H 3650 5950 60  0000 C CNN
-F 3 "" H 3650 5950 60  0000 C CNN
-	1    3650 5950
-	1    0    0    -1
-$EndComp
-Text Notes 2850 5600 0    60   ~ 0
+P 3650 6300
+F 0 "XP?" H 3900 6400 60  0000 C CNN
+F 1 "CONN_02_M" H 4000 6100 60  0001 C CNN
+F 2 "" H 3650 6300 60  0000 C CNN
+F 3 "" H 3650 6300 60  0000 C CNN
+	1    3650 6300
+	1    0    0    -1
+$EndComp
+Text Notes 2850 5950 0    60   ~ 0
 Connectors
 $Comp
 L PAD XS?
 U 1 1 55DA139F
-P 2850 6400
-F 0 "XS?" H 3100 6500 60  0000 C CNN
-F 1 "PAD" H 3100 6300 60  0000 C CNN
-F 2 "" H 2850 6400 60  0000 C CNN
-F 3 "" H 2850 6400 60  0000 C CNN
-	1    2850 6400
-	1    0    0    -1
-$EndComp
-$Comp
-L NMOS_Circle VT?
-U 1 1 55DAE0AB
-P 4300 5300
-F 0 "VT?" H 4400 5150 60  0000 R CNN
-F 1 "NMOS_Circle" H 4650 5500 60  0000 R CNN
-F 2 "" H 4275 5325 60  0000 C CNN
-F 3 "" H 4275 5325 60  0000 C CNN
-	1    4300 5300
-	1    0    0    -1
-$EndComp
-$Comp
-L PMOS_Circle VT?
-U 1 1 55DAE216
-P 5000 5300
-F 0 "VT?" H 5100 5150 60  0000 R CNN
-F 1 "PMOS_Circle" H 5350 5500 60  0000 R CNN
-F 2 "" H 4975 5325 60  0000 C CNN
-F 3 "" H 4975 5325 60  0000 C CNN
-	1    5000 5300
+P 2850 6750
+F 0 "XS?" H 3100 6850 60  0000 C CNN
+F 1 "PAD" H 3100 6650 60  0000 C CNN
+F 2 "" H 2850 6750 60  0000 C CNN
+F 3 "" H 2850 6750 60  0000 C CNN
+	1    2850 6750
 	1    0    0    -1
 $EndComp
@@
 L NPN_Circle VT?
 U 1 1 55DB069D
-P 3050 5250
-F 0 "VT?" H 3025 5100 60  0000 R CNN
-F 1 "NPN_Circle" H 3050 5400 60  0000 R CNN
-F 2 "" H 3050 5250 60  0000 C CNN
-F 3 "" H 3050 5250 60  0000 C CNN
-	1    3050 5250
+P 4350 4000
+F 0 "VT?" H 4325 3850 60  0000 R CNN
+F 1 "NPN_Circle" H 4350 4150 60  0000 R CNN
+F 2 "" H 4350 4000 60  0000 C CNN
+F 3 "" H 4350 4000 60  0000 C CNN
+	1    4350 4000
 	1    0    0    -1
 $EndComp
@@
 L PNP_Circle VT?
 U 1 1 55DB0714
-P 3700 5250
-F 0 "VT?" H 3675 5100 60  0000 R CNN
-F 1 "PNP_Circle" H 3700 5400 60  0000 R CNN
-F 2 "" H 3700 5250 60  0000 C CNN
-F 3 "" H 3700 5250 60  0000 C CNN
-	1    3700 5250
+P 5000 4000
+F 0 "VT?" H 4975 3850 60  0000 R CNN
+F 1 "PNP_Circle" H 5000 4150 60  0000 R CNN
+F 2 "" H 5000 4000 60  0000 C CNN
+F 3 "" H 5000 4000 60  0000 C CNN
+	1    5000 4000
 	1    0    0    -1
 $EndComp
@@
 	1    0    0    -1
 $EndComp
+$Comp
+L NJFET_Circle VT?
+U 1 1 55E24B68
+P 4400 4500
+F 0 "VT?" H 4475 4325 60  0000 R CNN
+F 1 "NJFET_Circle" H 4700 4675 60  0000 R CNN
+F 2 "" H 4350 4525 60  0000 C CNN
+F 3 "" H 4350 4525 60  0000 C CNN
+	1    4400 4500
+	1    0    0    -1
+$EndComp
+$Comp
+L NJFET VT?
+U 1 1 55E266D1
+P 3050 4500
+F 0 "VT?" H 3125 4350 60  0000 R CNN
+F 1 "NJFET" H 3175 4650 60  0000 R CNN
+F 2 "" H 3000 4525 60  0000 C CNN
+F 3 "" H 3000 4525 60  0000 C CNN
+	1    3050 4500
+	1    0    0    -1
+$EndComp
+$Comp
+L PJFET_Circle VT?
+U 1 1 55E2BB66
+P 5050 4500
+F 0 "VT?" H 5100 4325 60  0000 R CNN
+F 1 "PJFET_Circle" H 5325 4675 60  0000 R CNN
+F 2 "" H 4975 4525 60  0000 C CNN
+F 3 "" H 4975 4525 60  0000 C CNN
+	1    5050 4500
+	1    0    0    -1
+$EndComp
+$Comp
+L PJFET VT?
+U 1 1 55E2BDD2
+P 3700 4500
+F 0 "VT?" H 3775 4350 60  0000 R CNN
+F 1 "PJFET" H 3825 4650 60  0000 R CNN
+F 2 "" H 3625 4525 60  0000 C CNN
+F 3 "" H 3625 4525 60  0000 C CNN
+	1    3700 4500
+	1    0    0    -1
+$EndComp
+$Comp
+L PMOSFET_DE VT?
+U 1 1 55E38F96
+P 3700 5600
+F 0 "VT?" H 3775 5475 60  0000 R CNN
+F 1 "PMOSFET_DE" H 4000 5775 60  0000 R CNN
+F 2 "" H 3650 5625 60  0000 C CNN
+F 3 "" H 3650 5625 60  0000 C CNN
+	1    3700 5600
+	1    0    0    -1
+$EndComp
+$Comp
+L PMOSFET_DE_Circle VT?
+U 1 1 55E398A7
+P 5050 5600
+F 0 "VT?" H 5125 5450 60  0000 R CNN
+F 1 "PMOSFET_DE_Circle" H 5075 5800 60  0000 C CNN
+F 2 "" H 5000 5625 60  0000 C CNN
+F 3 "" H 5000 5625 60  0000 C CNN
+	1    5050 5600
+	1    0    0    -1
+$EndComp
+$Comp
+L NMOSFET_DE VT?
+U 1 1 55E3A2F0
+P 3050 5600
+F 0 "VT?" H 3125 5475 60  0000 R CNN
+F 1 "NMOSFET_DE" H 3050 5775 60  0000 C CNN
+F 2 "" H 3000 5625 60  0000 C CNN
+F 3 "" H 3000 5625 60  0000 C CNN
+	1    3050 5600
+	1    0    0    -1
+$EndComp
+$Comp
+L NMOSFET_DE_Circle VT?
+U 1 1 55E3A4D0
+P 4400 5600
+F 0 "VT?" H 4475 5450 60  0000 R CNN
+F 1 "NMOSFET_DE_Circle" H 4400 5900 60  0000 C CNN
+F 2 "" H 4350 5625 60  0000 C CNN
+F 3 "" H 4350 5625 60  0000 C CNN
+	1    4400 5600
+	1    0    0    -1
+$EndComp
+$Comp
+L NMOSFET VT?
+U 1 1 55E30D52
+P 3050 5050
+F 0 "VT?" H 3125 4925 60  0000 R CNN
+F 1 "NMOSFET" H 3050 5225 60  0000 C CNN
+F 2 "" H 3000 5075 60  0000 C CNN
+F 3 "" H 3000 5075 60  0000 C CNN
+	1    3050 5050
+	1    0    0    -1
+$EndComp
+$Comp
+L NMOSFET_Circle VT?
+U 1 1 55E30F2D
+P 4400 5050
+F 0 "VT?" H 4475 4900 60  0000 R CNN
+F 1 "NMOSFET_Circle" H 4400 5350 60  0000 C CNN
+F 2 "" H 4350 5075 60  0000 C CNN
+F 3 "" H 4350 5075 60  0000 C CNN
+	1    4400 5050
+	1    0    0    -1
+$EndComp
+$Comp
+L PMOSFET VT?
+U 1 1 55E3119D
+P 3700 5050
+F 0 "VT?" H 3775 4925 60  0000 R CNN
+F 1 "PMOSFET" H 3700 5225 60  0000 C CNN
+F 2 "" H 3650 5075 60  0000 C CNN
+F 3 "" H 3650 5075 60  0000 C CNN
+	1    3700 5050
+	1    0    0    -1
+$EndComp
+$Comp
+L PMOSFET_Circle VT?
+U 1 1 55E31284
+P 5050 5050
+F 0 "VT?" H 5125 4900 60  0000 R CNN
+F 1 "PMOSFET_Circle" H 5050 5250 60  0000 C CNN
+F 2 "" H 5000 5075 60  0000 C CNN
+F 3 "" H 5000 5075 60  0000 C CNN
+	1    5050 5050
+	1    0    0    -1
+$EndComp

Commit message: Add photo diode and diode bridge
Parts:
- removed HL?: LED, symbol LED
- added HL?: LED, symbol LED
- added VD?: Diode_Bridge, symbol Diode_Bridge
- added VD?: Photo_Diode, symbol Photo_Diode
Other:
- moved on the sheet: VT?, XP?, XS?
